File: AxxSolder_hardware/AxxSolder.kicad_pcb (KiCad board)
At the start: 2 copper layers, 39 x 82.5 mm, 147 parts, among them IC1 TLV76733DRVR, IC2 OPA2387DSGT, IC3 LMR54406DBVR, IC4 STM32G431CBT6, IC5 TPD4E1U06DBVR, IC6 STUSB4500QTR, IC7 MAX16171ATA_VY+T, IC8 LTC4440AHMS8E, IC9 INA281A5QDBVRQ1, J1 USB4110-GF-A, J2 691243110009, J3 TSW-102-07-T-S, J4 61300611821, J5 TSW-102-07-T-S, J6 TSW-102-07-T-S, J7 TSW-108-07-T-S, Q1 STL9P3LLH6, Q2 STL10N3LLH5, Q3 2N7002NXAKR, U2 PEC11J-9215F-S0015, U3 BSC014N04LS

Commit message: ordered
Parts:
- C10, C11, C34, C35, C5: footprint Capacitor_SMD:C_0603_1608Metric -> Capacitor_SMD:C_0805_2012Metric
- moved C35 1.28 mm to (183.5, 75.0)
- moved C34 0.50 mm to (183.0, 77.0)
- moved C10 0.25 mm to (191.2, 143.4)
- moved C11 0.25 mm to (189.7, 139.0)
- moved C5 0.13 mm to (169.5, 77.1)
Routing:
- net GND: track 435.4 -> 438.2 mm, vias 176 -> 182
- net VDD: track 58.8 -> 60.4 mm
- net /VBUS: track 33.2 -> 34.1 mm
- net Net-(IC3-FB): track 16.4 -> 17.4 mm
- net Net-(R46-Pad2): track 20.8 -> 21.4 mm
Other:
- board text added: "2026-11"
- board text added: "Modded by Cseka"
- board text added: "V3.2c"
- board text added: "WHEN TIP GROUNDING IS REQUIRED: USE A SUPPLY WITH FLOATING OUT NOT GROUNDED USB CONNECTION"
- board text removed: "2025-03"
- board text removed: "V3.2"
- board text removed: "WHEN TIP GROUNDING IS REQUIRED: USE A SUPPLY WITH FLOATING OUTPUT (SELV) NO GROUNDED USB CONNECTION"
