File: AxxSolder_hardware/AxxSolder.kicad_sch (KiCad schematic)
At the start: 152 parts, among them IC1 TLV76733DRVR, IC2 OPA2387DSGT, IC3 LMR54406DBVR, IC4 STM32G431CBT6, IC5 TPD4E1U06DBVR, IC6 STUSB4500QTR, IC7 MAX16171ATA_VY+T, IC8 LTC4440AHMS8E, IC9 INA281A5QDBVRQ1, J1 USB4110-GF-A, J2 691243110009, J3 TSW-102-07-T-S, J4 61300611821, J5 TSW-102-07-T-S, J6 TSW-102-07-T-S, J7 TSW-108-07-T-S, J8 Conn_01x01_Pin, Q1 STL9P3LLH6, Q2 STL10N3LLH5, Q3 2N7002NXAKR, U2 PEC11J-9215F-S0015, U3 BSC014N04LS

Commit message: ordered
Parts:
- C1, C12, C13, C19, C2, C20, C30, C31, C32, C7, C8: value 10u -> 10u 16V
- C10, C11, C34, C35, C5: value 10u -> 10u 35V; footprint Capacitor_SMD:C_0603_1608Metric -> Capacitor_SMD:C_0805_2012Metric; Manufacturer_Name Murata Electronics -> (none); Manufacturer_Part_Number GRM188R6YA106MA73J -> (none); Mouser Part Number 81-GRM188R6YA106MA3J -> (none)
- TFT1: value ~ -> (none)
